Commit message: xacro gazebo

File: f1tenth_gym_ros/launch/gazebo_racecar.xacro (robot description, xacro)
@@ -303,7 +303,4 @@
     <mu2>${wheel_mu2}</mu2>
   </gazebo>
-  <gazebo reference="${car_name}/laser_model">
-    <material>Gazebo/Black</material>
-  </gazebo>
   <!-- Propiedades de Gazebo para la cámara depth -->
   <gazebo reference="${car_name}/camera_link">
@@ -342,3 +339,39 @@
     </sensor>
   </gazebo>
+  <gazebo reference="${car_name}/laser_model">
+    <material>Gazebo/Black</material>
+    <sensor type="ray" name="hokuyo">
+      <pose>0 0 0 0 0 0</pose>
+      <visualize>true</visualize>
+      <update_rate>40</update_rate>
+      <ray>
+        <scan>
+          <horizontal>
+            <samples>720</samples>
+            <resolution>1</resolution>
+            <min_angle>-3.141593</min_angle>
+            <max_angle>3.141593</max_angle>
+          </horizontal>
+        </scan>
+        <range>
+          <min>0.10</min>
+          <max>30.0</max>
+          <resolution>0.01</resolution>
+        </range>
+        <noise>
+          <type>gaussian</type>
+          <mean>0.0</mean>
+          <stddev>0.01</stddev>
+        </noise>
+      </ray>
+      <plugin name="gazebo_ros_head_hokuyo_controller" filename="libgazebo_ros_ray_sensor.so">
+        <ros>
+          <namespace></namespace>
+          <remapping>~/out:=scan</remapping>
+        </ros>
+        <output_type>sensor_msgs/LaserScan</output_type>
+        <frame_name>ego_racecar/laser_model</frame_name>
+      </plugin>
+    </sensor>
+  </gazebo>
 </robot>
